Commit message: revolute -> fixed test

File: dofbot_moveit/urdf/dofbot_isaac_mimic_all.urdf (robot description, URDF)
Before this commit: robot yahboom_dofbot, 12 links, 11 joints
Joints:
- joint llink_joint3: axis 0 0 1 -> (none); limit lower=-1.54 upper=0 effort=100 velocity=1 -> (none); mimic joint=grip_joint multiplier=-1 offset=0 -> (none); type revolute -> fixed
- joint rlink_joint3: axis 0 0 1 -> (none); limit lower=-1.54 upper=0 effort=100 velocity=1 -> (none); mimic joint=grip_joint multiplier=1 offset=0 -> (none); type revolute -> fixed

Commit message: loop 생성

File: dofbot_moveit/urdf/dofbot_isaac_mimic_all.urdf (robot description, URDF)
Before this commit: robot yahboom_dofbot, 12 links, 11 joints
Joints:
- joint llink_joint3: axis (none) -> 0 0 1; limit (none) -> lower=-1.54 upper=0 effort=100 velocity=1; mimic (none) -> joint=grip_joint multiplier=-1 offset=0; type fixed -> revolute
- joint rlink_joint3: axis (none) -> 0 0 1; limit (none) -> lower=-1.54 upper=0 effort=100 velocity=1; mimic (none) -> joint=grip_joint multiplier=1 offset=0; type fixed -> revolute
