Commit message: urdf 수정

File: gazebo_yahboom_dofbot.urdf (robot description, URDF)
Before this commit: robot yahboom_dofbot, 12 links, 11 joints
Links:
- link llink1: geometry collision mesh filename=package://yahboomcar_description/meshes/X3plus/visual/llink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; visual mesh filename=package://yahboomcar_description/meshes/X3plus/visual/llink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
- link llink2: geometry collision mesh filename=package://yahboomcar_description/meshes/X3plus/visual/llink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; visual mesh filename=package://yahboomcar_description/meshes/X3plus/visual/llink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
- link llink3: geometry collision mesh filename=package://yahboomcar_description/meshes/X3plus/visual/llink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; visual mesh filename=package://yahboomcar_description/meshes/X3plus/visual/llink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
- link rlink1: geometry collision mesh filename=package://yahboomcar_description/meshes/X3plus/visual/rlink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; visual mesh filename=package://yahboomcar_description/meshes/X3plus/visual/rlink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
- link rlink2: geometry collision mesh filename=package://yahboomcar_description/meshes/X3plus/visual/rlink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; visual mesh filename=package://yahboomcar_description/meshes/X3plus/visual/rlink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
- link rlink3: geometry collision mesh filename=package://yahboomcar_description/meshes/X3plus/visual/rlink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; visual mesh filename=package://yahboomcar_description/meshes/X3plus/visual/rlink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
